Commit message: add dummy intertia for gazebo

File: zed_description/urdf/zed_macro.urdf.xacro (robot description, xacro)
@@ -73,5 +73,11 @@
     </xacro:if>
     <!-- Camera mounting point (the threaded screw hole in the bottom) -->
-    <link name="${name}_camera_link" />
+    <link name="${name}_camera_link">
+      <inertial>
+        <origin xyz= "0 0 0" rpy = "0 0 0" />
+        <mass value="1.0" />
+        <inertia ixx="0.1" ixy="0.0" ixz="0.0" iyy="0.1" iyz="0.0" izz="0.1"/>
+      </inertial>
+    </link>
     <!-- Camera Center -->
     <link name="${name}_camera_center">
